File: Sailowtech/Sailowtech.kicad_pcb (KiCad board)
At the start: 2 copper layers, 110.5 x 110 mm, 12 parts, among them J1 Second Board Connector, U1 Zigbee, U2 ESP32-DEVKITM-1

Commit message: Rond m190
Parts:
- moved I2C_3.3V_GND_SDA_SCL2 269.7 mm to (-4.00, -83.0), turned to 180 degrees
- moved GPS1 213.5 mm to (0.50, -49.0), turned to 180 degrees
- moved MicroSD1 211.4 mm to (-55.5, 11.2), turned to 0 degrees
- moved U2 198.6 mm to (0.57, -0.33)
- moved Logic_level_Converter1 189.2 mm to (-32.9, 35.1), turned to 180 degrees
- moved J1 164.7 mm to (80.4, 0.96)
- moved U1 163.4 mm to (-30.4, 0.12), turned to 0 degrees
- moved CAN_Trans1 163.2 mm to (-19.1, 45.6), turned to 180 degrees
- moved I2C_3.3V_GND_SDA_SCL1 159.1 mm to (19.0, -83.0)
- moved NMEA1 127.4 mm to (-12.5, 82.5), turned to 0 degrees
- moved LM2596 121.7 mm to (16.2, 50.4)
- moved Battery1 105.3 mm to (13.0, 82.2), turned to 0 degrees
Routing:
- net +3.3V: track 210.8 -> 388.4 mm
- net +5V: track 227.3 -> 374.6 mm
- net Net-(U1-RX/D7): track 71.6 -> 12.9 mm
- net Net-(U1-TX/D6): track 83.7 -> 27.9 mm
- net Net-(U2-GPIO2): track 23.6 -> 74.1 mm
- net Net-(U2-GPIO13): track 24.7 -> 74.9 mm
- net Net-(U2-GPIO12): track 25.2 -> 74.7 mm
- net Net-(U2-GPIO15): track 24.2 -> 73.5 mm
- net /SCL: track 151.4 -> 198.8 mm
- net Net-(LM2596-3.2-40V): track 15.6 -> 55.7 mm
- net Net-(MicroSD1-CS): track 34.7 -> 69.1 mm
- net Net-(GPS1-TX): track 17.3 -> 50.8 mm
- net Net-(GPS1-RX): track 20.8 -> 54.3 mm
- net Net-(Logic_level_Converter1-LV2): track 15.1 -> 46.1 mm
- net Net-(MicroSD1-D1): track 38.3 -> 69.1 mm
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Other:
- board size 110.5 x 110 mm -> 190 x 190 mm

Commit message: SecondBoard Rond m130
Parts:
- removed I2C_3.3V_GND_SDA_SCL1, I2C_3.3V_GND_SDA_SCL2: ~, TerminalBlock_Phoenix:TerminalBlock_Phoenix_MKDS-1,5-4_1x04_P5.00mm_Horizontal
- moved Battery1 78.1 mm to (54.4, 16.0), turned to 90 degrees
- moved CAN_Trans1 67.4 mm to (43.9, 21.8), turned to 0 degrees
- moved Logic_level_Converter1 63.4 mm to (30.3, 30.1)
- moved LM2596 43.8 mm to (-26.9, 42.7)
- moved MicroSD1 40.2 mm to (-21.6, -10.4)
- moved J1 27.8 mm to (53.3, -5.33)
- moved NMEA1 27.8 mm to (-7.40, 55.2)
- moved U1 11.0 mm to (-37.4, 8.65)
- moved U2 8.16 mm to (0.07, -8.46)
- moved GPS1 1.02 mm to (0.14, -50.0), turned to -90 degrees
Routing:
- net +3.3V: track 388.4 -> 177.0 mm
- net GND: track 463.2 -> 290.4 mm
- net +5V: track 374.6 -> 221.7 mm
- net /SCL: track 198.8 -> 59.5 mm
- net /SDA: track 204.5 -> 68.8 mm
- net Net-(CAN_Trans1-CANL): track 26.9 -> 82.1 mm
- net Net-(CAN_Trans1-CANH): track 31.5 -> 77.4 mm
- net Net-(MicroSD1-D1): track 69.1 -> 37.1 mm
- net Net-(MicroSD1-D0): track 69.1 -> 37.1 mm
- net Net-(MicroSD1-SCK): track 69.1 -> 37.1 mm
- net Net-(MicroSD1-CS): track 69.1 -> 37.1 mm
- net Net-(U2-GPIO13): track 74.9 -> 46.7 mm
- net Net-(U2-GPIO2): track 74.1 -> 46.2 mm
- net Net-(U2-GPIO12): track 74.7 -> 47.2 mm
- net Net-(U2-GPIO15): track 73.5 -> 46.2 mm
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Other:
- board size 190 x 190 mm -> 130 x 130 mm

Commit message: Plan de masse Update
Connections:
- J1 pad 10: /SDA -> Net-(U2-GPIO21)
- J1 pad 8: /SCL -> Net-(U2-GPIO22)
- U2 pad J1_10: /SDA -> unconnected-(U2-GPIO32-PadJ1_10)
- U2 pad J1_11: /SCL -> unconnected-(U2-GPIO33-PadJ1_11)
- U2 pad J3_4: /SDA -> Net-(U2-GPIO21)
- U2 pad J3_5: /SCL -> Net-(U2-GPIO22)
Routing:
- net GND: track 290.4 -> 0.22 mm
- net +5V: track 221.7 -> 382.7 mm
- net /SDA: track 68.8 -> 0.00 mm
- net Net-(U2-GPIO21): track 0.00 -> 68.8 mm
- net Net-(U2-GPIO22): track 0.00 -> 59.5 mm
- net /SCL: track 59.5 -> 0.00 mm
- net Net-(LM2596-3.2-40V): track 68.5 -> 64.1 mm
- added copper zone on B.Cu, net GND

Commit message: changement connecteur
Parts:
- removed J1: Second Board Connector, M50-3550542:HARWIN_M50-3550542
- added J2: Conn_01x10_Socket, Connector_PinHeader_2.54mm:PinHeader_1x10_P2.54mm_Vertical, B.Cu at (55.0, -11.4)
- Battery1: footprint TerminalBlock_Phoenix:TerminalBlock_Phoenix_MKDS-1,5-2_1x02_P5.00mm_Horizontal -> Connector_Phoenix_MC:PhoenixContact_MCV_1,5_2-G-3.5_1x02_P3.50mm_Vertical
- NMEA1: footprint TerminalBlock_Phoenix:TerminalBlock_Phoenix_MKDS-1,5-4_1x04_P5.00mm_Horizontal -> Connector_Phoenix_MC:PhoenixContact_MCV_1,5_4-G-3.5_1x04_P3.50mm_Vertical
- moved Battery1 58.0 mm to (10.3, 53.6), turned to 0 degrees
- moved NMEA1 4.28 mm to (-11.5, 54.0)
- moved U1 1.86 mm to (-38.9, 7.62), turned to 90 degrees
Routing:
- net Net-(U1-RX/D7): track 24.4 -> 74.6 mm
- net +5V: track 382.7 -> 408.0 mm
- net Net-(J2-Pin_5): track 68.8 -> 51.7 mm
- net Net-(U1-TX/D6): track 40.7 -> 26.6 mm
- net Net-(LM2596-3.2-40V): track 64.1 -> 53.4 mm
- net Net-(J2-Pin_6): track 59.5 -> 51.7 mm
- net Net-(CAN_Trans1-CANH): track 77.4 -> 82.0 mm
- net Net-(CAN_Trans1-CANL): track 82.1 -> 85.7 mm
- net +3.3V: track 177.0 -> 178.6 mm
- net Net-(J2-Pin_8): track 46.2 -> 47.4 mm
- net Net-(J2-Pin_7): track 46.2 -> 47.2 mm
- net Net-(J2-Pin_9): track 46.7 -> 47.7 mm
- net Net-(J2-Pin_10): track 47.2 -> 47.8 mm
Other:
- outline, holes or cut-outs redrawn

Commit message: finished version
Changed lines of the file:
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@@
 			(outputformat 1)
 			(mirror no)
-			(drillshape 1)
+			(drillshape 0)
 			(scaleselection 1)
-			(outputdirectory "")
+			(outputdirectory "Gerber")
 		)
 	)
@@
 		(polygon
 			(pts
-				(xy -58.5 -69.5) (xy -82.5 59) (xy 80.5 77.5) (xy 98 -111.5)
+				(xy -120.5 -101) (xy -98 80.5) (xy 132.5 107) (xy 150.5 -104)
 			)
 		)
